Commit message: Add 1st and 2nd links

File: urdf/arm.urdf (robot description, URDF)
Before this commit: robot arm, 1 links, 0 joints
Links:
- added link link_1; visual cylinder length=0.05 radius=0.02
- added link link_2; visual cylinder length=0.05 radius=0.02
- link base_link: geometry visual cylinder length=0.05 radius=0.05
Joints:
- added joint 1_to_2: type revolute, parent link_1, child link_2, origin xyz=0 0 0.05, axis 0 1 0, limit lower=0.0 upper=1.548 effort=1000.0 velocity=0.5
- added joint base_to_1: type continuous, parent base_link, child link_1, origin xyz=0 0 0.05, axis 0 0 1
